File: Capteur_graphique_Final/Capteur_Graphite/Capteur_Graphite.kicad_pcb (KiCad board)
At the start: 2 copper layers, 68.6 x 53.3 mm, 24 parts, among them J1 Power, J2 Digital/PWM, J3 Analog, J4 Digital/PWM, U2 MCP41050, U7 LTC1050ACN8_PBF

Commit message: Modifs de Vicky pendant les vacances
Parts:
- R6: value 47k -> 33k
- moved C3 12.4 mm to (151.6, 71.2), turned to -90 degrees
- moved C2 2.40 mm to (144.8, 92.6)
- moved R5 2.31 mm to (108.4, 76.8)
- moved U3 2.10 mm to (155.6, 63.8)
Connections:
- C3 pad 1: +5V -> D2
- J2 pad 10: /8 -> D8
- J4 pad 1: /7 -> D7
- J4 pad 7: D1 -> /TX/1
- J4 pad 8: D0 -> /RX/0
- U3 pad 3: D0 -> D8
- U3 pad 4: D1 -> D7
Routing:
- net +5V: track 202.6 -> 132.4 mm
- net D7: track 0.00 -> 32.7 mm, vias 0 -> 2
- net D8: track 0.00 -> 32.6 mm, vias 0 -> 2
- net D0: track 15.4 -> 0.00 mm
- net D1: track 10.9 -> 0.00 mm
- net D2: track 24.9 -> 29.2 mm
- net Net-(U7-+IN): track 18.1 -> 16.4 mm
- net Net-(U6-OUT): track 4.86 -> 3.35 mm
Other:
- board size 68.6 x 53.3 mm -> 68.6 x 53.4 mm
