File: Capteur_graphique_Final/Capteur_Graphite/Capteur_Graphite.kicad_sch (KiCad schematic)
At the start: 20 parts, among them J1 Power, J2 Digital/PWM, J3 Analog, J4 Digital/PWM, U2 MCP41050, U7 LTC1050ACN8_PBF

Commit message: Modifs de Vicky pendant les vacances
Parts:
- R6: value 47k -> 33k
Connections:
- net +5V: no longer C3.1
- net D2: now also C3.1
- net 7 renamed D7
- net D7: now also U3.4 (RX)
- net 8 renamed D8
- net D8: now also U3.3 (TX)
- net D0 renamed RX/0
- net RX/0: no longer U3.3 (TX)
- net D1 renamed TX/1
- net TX/1: no longer U3.4 (RX)
- no-connect marks 13 -> 20
Changed lines of the file:
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@@
 	)
 	(junction
-		(at 259.08 59.69)
+		(at 240.03 82.55)
 		(diameter 0)
 		(color 0 0 0 0)
 	)
 	(junction
-		(at 240.03 82.55)
+		(at 231.14 53.34)
 		(diameter 0)
 		(color 0 0 0 0)
 	)
 	(junction
-		(at 231.14 53.34)
+		(at 129.54 82.55)
 		(diameter 0)
 		(color 0 0 0 0)
 	)
 	(junction
-		(at 129.54 82.55)
+		(at 158.75 165.1)
 		(diameter 0)
 		(color 0 0 0 0)
@@
 		(color 0 0 0 0)
 	)
+	(junction
+		(at 151.13 176.53)
+		(diameter 0)
+		(color 0 0 0 0)
+	)
 	(no_connect
 		(at 21.59 64.77)
@@
 	)
 	(no_connect
-		(at 74.93 59.69)
+		(at 222.25 92.71)
+	)
+	(no_connect
+		(at 222.25 95.25)
+	)
+	(no_connect
+		(at 222.25 97.79)
+	)
+	(no_connect
+		(at 77.47 62.23)
+	)
+	(no_connect
+		(at 222.25 85.09)
+	)
+	(no_connect
+		(at 77.47 69.85)
 	)
 	(no_connect
@@
 	)
 	(no_connect
-		(at 74.93 62.23)
+		(at 78.74 77.47)
 	)
 	(no_connect
@@
 	)
 	(no_connect
+		(at 222.25 87.63)
+	)
+	(no_connect
+		(at 222.25 90.17)
+	)
+	(no_connect
+		(at 78.74 74.93)
+	)
+	(no_connect
 		(at 19.05 34.29)
 	)
@@
 	)
 	(no_connect
-		(at 74.93 49.53)
+		(at 222.25 100.33)
 	)
 	(no_connect
@@
 	)
 	(no_connect
-		(at 74.93 69.85)
-	)
-	(no_connect
 		(at 74.93 29.21)
 	)
@@
 	(wire
 		(pts
-			(xy 259.08 67.31) (xy 259.08 71.12)
+			(xy 158.75 165.1) (xy 160.02 165.1)
 		)
 		(stroke
@@
 	(wire
 		(pts
+			(xy 156.21 176.53) (xy 151.13 176.53)
+		)
+		(stroke
+			(width 0)
+			(type default)
+		)
+	)
+	(wire
+		(pts
 			(xy 149.86 53.34) (xy 149.86 80.01)
 		)
@@
 	(wire
 		(pts
-			(xy 62.23 59.69) (xy 74.93 59.69)
+			(xy 62.23 59.69) (xy 77.47 59.69)
 		)
 		(stroke
@@
 	(wire
 		(pts
-			(xy 62.23 62.23) (xy 74.93 62.23)
+			(xy 62.23 62.23) (xy 77.47 62.23)
 		)
 		(stroke
@@
 	(wire
 		(pts
-			(xy 151.13 175.26) (xy 151.13 177.8)
+			(xy 158.75 165.1) (xy 158.75 171.45)
+		)
+		(stroke
+			(width 0)
+			(type default)
+		)
+	)
+	(wire
+		(pts
+			(xy 151.13 175.26) (xy 151.13 176.53)
 		)
 		(stroke
@@
 	(wire
 		(pts
+			(xy 158.75 171.45) (xy 163.83 171.45)
+		)
+		(stroke
+			(width 0)
+			(type default)
+		)
+	)
+	(wire
+		(pts
+			(xy 163.83 179.07) (xy 156.21 179.07)
+		)
+		(stroke
+			(width 0)
+			(type default)
+		)
+	)
+	(wire
+		(pts
 			(xy 166.37 80.01) (xy 149.86 80.01)
 		)
@@
 	(wire
 		(pts
+			(xy 156.21 179.07) (xy 156.21 176.53)
+		)
+		(stroke
+			(width 0)
+			(type default)
+		)
+	)
+	(wire
+		(pts
 			(xy 58.42 139.7) (xy 58.42 143.51)
 		)
@@
 	(wire
 		(pts
+			(xy 151.13 176.53) (xy 151.13 177.8)
+		)
+		(stroke
+			(width 0)
+			(type default)
+		)
+	)
+	(wire
+		(pts
 			(xy 149.86 80.01) (xy 149.86 93.98)
 		)
@@
 	(wire
 		(pts
+			(xy 167.64 176.53) (xy 168.91 176.53)
+		)
+		(stroke
+			(width 0)
+			(type default)
+		)
+	)
+	(wire
+		(pts
 			(xy 17.78 72.39) (xy 34.29 72.39)
 		)
@@
 	(wire
 		(pts
-			(xy 62.23 69.85) (xy 74.93 69.85)
+			(xy 62.23 69.85) (xy 77.47 69.85)
 		)
 		(stroke
@@
 	(wire
 		(pts
-			(xy 144.78 165.1) (xy 152.4 165.1)
+			(xy 144.78 165.1) (xy 158.75 165.1)
 		)
 		(stroke
@@
 		)
 	)
-	(global_label "D0"
+	(global_label "D7"
 		(shape input)
-		(at 78.74 77.47 0)
+		(at 77.47 59.69 0)
 		(fields_autoplaced yes)
 		(effects
@@
 		)
 		(property "Intersheetrefs" "${INTERSHEET_REFS}"
-			(at 84.2998 77.47 0)
+			(at 83.0298 59.69 0)
 			(effects
 				(font
@@
 		)
 	)
-	(global_label "D1"
+	(global_label "D8"
 		(shape input)
-		(at 78.74 74.93 0)
+		(at 74.93 49.53 0)
 		(fields_autoplaced yes)
 		(effects
@@
 		)
 		(property "Intersheetrefs" "${INTERSHEET_REFS}"
-			(at 84.2998 74.93 0)
+			(at 80.4898 49.53 0)
 			(effects
 				(font
@@
 		)
 	)
-	(global_label "D0"
+	(global_label "D8"
 		(shape input)
 		(at 41.91 143.51 90)
@@
 		)
 	)
-	(global_label "D1"
+	(global_label "D7"
 		(shape input)
 		(at 44.45 143.51 90)
@@
 	(global_label "D2"
 		(shape input)
-		(at 152.4 165.1 0)
+		(at 160.02 165.1 0)
 		(fields_autoplaced yes)
 		(effects
@@
 		)
 		(property "Intersheetrefs" "${INTERSHEET_REFS}"
-			(at 157.9598 165.1 0)
+			(at 165.5798 165.1 0)
 			(effects
 				(font
@@
 			)
 		)
-		(property "Value" "47k"
+		(property "Value" "33k"
 			(at 138.43 128.27 90)
 			(effects
@@
 	)
 	(symbol
-		(lib_name "GND_9")
-		(lib_id "power:GND")
-		(at 259.08 71.12 0)
-		(unit 1)
-		(exclude_from_sim no)
-		(in_bom yes)
-		(on_board yes)
-		(dnp no)
-		(fields_autoplaced yes)
-		(property "Reference" "#PWR021"
-			(at 259.08 77.47 0)
-			(effects
-				(font
-					(size 1.27 1.27)
-				)
-				(hide yes)
-			)
-		)
-		(property "Value" "GND"
-			(at 259.08 76.2 0)
-			(effects
-				(font
-					(size 1.27 1.27)
-				)
-			)
-		)
-		(property "Footprint" ""
-			(at 259.08 71.12 0)
-			(effects
-				(font
-					(size 1.27 1.27)
-				)
-				(hide yes)
-			)
-		)
-		(property "Datasheet" ""
-			(at 259.08 71.12 0)
-			(effects
-				(font
-					(size 1.27 1.27)
-				)
-				(hide yes)
-			)
-		)
-		(property "Description" "Power symbol creates a global label with name \"GND\" , ground"
-			(at 259.08 71.12 0)
-			(effects
-				(font
-					(size 1.27 1.27)
-				)
-				(hide yes)
-			)
-		)
-		(pin "1"
-		)
-		(instances
-			(project ""
-				(path "/e63e39d7-6ac0-4ffd-8aa3-1841a4541b55"
-					(reference "#PWR021")
-					(unit 1)
-				)
-			)
-		)
-	)
-	(symbol
 		(lib_id "Device:R")
 		(at 124.46 82.55 90)
@@
 	(symbol
 		(lib_id "Device:C")
-		(at 259.08 63.5 0)
+		(at 163.83 175.26 0)
 		(unit 1)
 		(exclude_from_sim no)
@@
 		(fields_autoplaced yes)
 		(property "Reference" "C3"
-			(at 262.89 62.2299 0)
+			(at 167.64 173.9899 0)
 			(effects
 				(font
@@
 		)
 		(property "Value" "100n"
-			(at 262.89 64.7699 0)
+			(at 167.64 176.5299 0)
 			(effects
 				(font
@@
 		)
 		(property "Footprint" "Capacitor_THT:C_Disc_D3.8mm_W2.6mm_P2.50mm"
-			(at 260.0452 67.31 0)
+			(at 164.7952 179.07 0)
 			(effects
 				(font
@@
 		)
 		(property "Datasheet" "~"
-			(at 259.08 63.5 0)
+			(at 163.83 175.26 0)
 			(effects
 				(font
@@
 		)
 		(property "Description" "Unpolarized capacitor"
-			(at 259.08 63.5 0)
+			(at 163.83 175.26 0)
 			(effects
 				(font
@@
 		)
 		(instances
-			(project "Capteur_Graphite"
+			(project ""
 				(path "/e63e39d7-6ac0-4ffd-8aa3-1841a4541b55"
 					(reference "C3")
